Commit message: joint leg origin

File: gong_ws/src/tf2_basic/urdf/02_leg_joint.urdf (robot description, URDF)
Before this commit: robot myfirst, 3 links, 2 joints
Links:
- removed link left_link
- added link left_leg; visual box size=0.6 0.1 0.2
Joints:
- joint base_to_left_leg: origin (none) -> xyz=0 0.22 0.25
- joint base_to_right_leg: origin (none) -> xyz=0 -0.22 0.25
