Commit message: pysics

File: gong_ws/src/tf2_basic/urdf/04_pysics.urdf (robot description, URDF)
Before this commit: robot visual, 16 links, 15 joints
Links:
- link right_gripper: geometry collision mesh filename=package://tf2_basic/meshes/l_finger.dae; visual mesh filename=package://tf2_basic/meshes/l_finger.dae
- link right_tip: geometry collision mesh filename=package://tf2_basic/meshes/l_finger_tip.dae; visual mesh filename=package://tf2_basic/meshes/l_finger_tip.dae
